File: extras/etapa_analogica_SigamDelta/etapa_analogica_SigmaDelta.kicad_pcb (KiCad board)
At the start: 2 copper layers, 63.5 x 78.8 mm, 17 parts, among them P1 CONN_02X10, P2 CONN_01X03, P3 CONN_02X10, P4 BNC

Commit message: Se agrega R5, R6 al layout
Parts:
- added R5: 1k, Resistors_SMD:R_0805_HandSoldering, F.Cu at (134.3, 89.5)
- added R6: 1k, Resistors_SMD:R_0805_HandSoldering, F.Cu at (125.5, 90.1)
- C3: value 220u -> 22u
- R1: value 1,2k -> 560
Connections:
- C3 pad 1: /N40 -> Net-(C3-Pad1)
- C6 pad 1: /N40 -> Net-(C6-Pad1)
- D1 pad 1: GND -> Net-(D1-Pad1)
- D1 pad 2: Net-(D1-Pad2) -> GND
- D1 pad 3: Net-(D1-Pad3) -> (no net)
- P1 pad 1: Net-(P1-Pad1) -> /5v
- P1 pad 10: Net-(P1-Pad10) -> /Tx
- P1 pad 12: /Rx -> Net-(P1-Pad12)
- P1 pad 14: /Tx -> Net-(P1-Pad14)
- P1 pad 3: Net-(P1-Pad3) -> /3.3v
- P1 pad 8: Net-(P1-Pad8) -> /Rx
- P2 pad 1: /Tx -> /Rx
- P2 pad 2: /Rx -> /Tx
- P3 pad 1: Net-(P3-Pad1) -> /5v
- R1 pad 1: Net-(D1-Pad2) -> Net-(D1-Pad1)
- R4 pad 1: /N40 -> Net-(C3-Pad1)
- RV1 pad 1: Net-(D1-Pad2) -> Net-(D1-Pad1)
- RV2 pad 2: Net-(R4-Pad2) -> Net-(RV2-Pad2)
